Commit message: change tool0 link

File: ur_description/urdf/inc/ur_macro.xacro (robot description, xacro)
@@ -312,5 +312,5 @@
     <joint name="${prefix}flange-tool0" type="fixed">
       <!-- default toolframe: X+ left, Y+ up, Z+ front -->
-      <origin xyz="0 0 0" rpy="${pi/2.0} 0 ${pi/2.0}"/>
+      <origin xyz="0.05 0.0 0.0" rpy="${pi/2.0} 0 ${pi/2.0}"/>
       <parent link="${prefix}flange"/>
       <child link="${prefix}tool0"/>

Commit message: adapt own work object

File: ur_description/urdf/inc/ur_macro.xacro (robot description, xacro)
@@ -312,5 +312,5 @@
     <joint name="${prefix}flange-tool0" type="fixed">
       <!-- default toolframe: X+ left, Y+ up, Z+ front -->
-      <origin xyz="0.05 0.0 0.0" rpy="${pi/2.0} 0 ${pi/2.0}"/>
+      <origin xyz="0.07 0.0 0.0" rpy="${pi/2.0} 0 ${pi/2.0}"/>
       <parent link="${prefix}flange"/>
       <child link="${prefix}tool0"/>

File: ur_gazebo/urdf/ur_macro.xacro (robot description, xacro)
@@ -47,4 +47,7 @@
     -->
     <xacro:include filename="$(find ur_description)/urdf/inc/ur_macro.xacro"/>
+    <xacro:include filename="$(find polsh_path_plan)/urdf/model_mount.xacro" />
+    <xacro:include filename="$(find polsh_path_plan)/urdf/kamaboko.xacro" />
+    <xacro:include filename="$(find polsh_path_plan)/urdf/kamaboko_outor.xacro" />
     <!-- Instantiate model for the REAL robot. -->
     <xacro:ur_robot
@@ -104,4 +107,7 @@
       </plugin>
     </gazebo>
+  <xacro:model_mount parent="wrist_3_link" prefix="mount_base" xyz = "0 0 0.00"/>
+  <xacro:kamaboko parent = "mount_base_link" prefix = "model" xyz = "0 0 0.07"/>
+  <xacro:kamaboko_outor parent = "model_link" prefix = "model_out" xyz = "0 0 0.00"/>
   </xacro:macro>
 </robot>

Commit message: change ee param

File: ur_description/urdf/inc/ur_macro.xacro (robot description, xacro)
@@ -312,5 +312,6 @@
     <joint name="${prefix}flange-tool0" type="fixed">
       <!-- default toolframe: X+ left, Y+ up, Z+ front -->
-      <origin xyz="0.07 0.0 0.0" rpy="${pi/2.0} 0 ${pi/2.0}"/>
+      <!-- <origin xyz="0.07 0.0 0.0" rpy="${pi/2.0} 0 ${pi/2.0}"/> -->
+      <origin xyz="${0.07+0.0375} 0.0 0.0" rpy="${pi/2.0} 0 ${pi/2.0}"/>
       <parent link="${prefix}flange"/>
       <child link="${prefix}tool0"/>

File: ur_description/urdf/ur.xacro (robot description, xacro)
@@ -35,5 +35,5 @@
      safety_k_position="$(arg safety_k_position)"/>
      <xacro:model_mount parent="wrist_3_link" prefix="mount_base" xyz = "0 0 0.00"/>
-     <xacro:kamaboko parent = "mount_base_link" prefix = "model" xyz = "0 0 0.07"/>
+     <xacro:kamaboko parent = "mount_base_link" prefix = "model" xyz = "0 0 ${0.07+0.0375}"/>
      <xacro:kamaboko_outor parent = "model_link" prefix = "model_out" xyz = "0 0 0.00"/>
      <xacro:sanding_machine parent = "base_link" prefix = "sand_origin" xyz = "-0.14147 ${0.643} 0.3"/>

File: ur_gazebo/urdf/ur_macro.xacro (robot description, xacro)
@@ -110,5 +110,5 @@
     </gazebo>
   <xacro:model_mount parent="wrist_3_link" prefix="mount_base" xyz = "0 0 0.00"/>
-  <xacro:kamaboko parent = "mount_base_link" prefix = "model" xyz = "0 0 0.07"/>
+  <xacro:kamaboko parent = "mount_base_link" prefix = "model" xyz = "0 0 ${0.07+0.0375}"/>
   <xacro:kamaboko_outor parent = "model_link" prefix = "model_out" xyz = "0 0 0.00"/>
   <xacro:sanding_machine parent = "base_link" prefix = "sand_origin" xyz = "-0.14147 0.643 0.3"/>
